File: TooManyKeys.kicad_pcb (KiCad board)
At the start: 6 copper layers, 156 x 116.5 mm, 82 parts

Commit message: Redo schematic references to match ergogen, work on connecting sch and pcb.
Routing:
- net R4: track 0.00 -> 7.00 mm, vias 0 -> 2
Changed lines of the file:
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@@
 		(pad "2" thru_hole circle
 			(at -0.915 0.55)
-			(size 0.45 0.45)
-			(drill 0.2)
+			(size 0.5 0.5)
+			(drill 0.3)
 			(layers "*.Cu" "*.Paste" "*.Mask")
 			(remove_unused_layers no)
@@
 		(net 41)
 	)
+	(via
+		(at 130.768327 173.357023)
+		(size 0.6)
+		(drill 0.3)
+		(layers "F.Cu" "B.Cu")
+		(net 42)
+	)
+	(via
+		(at 130.768327 166.357023)
+		(size 0.6)
+		(drill 0.3)
+		(layers "F.Cu" "B.Cu")
+		(net 42)
+	)
+	(segment
+		(start 130.768327 173.357023)
+		(end 130.768327 166.357023)
+		(width 0.2)
+		(layer "In3.Cu")
+		(net 42)
+	)
 	(embedded_fonts no)
