File: toomanykeys_right.kicad_pcb (KiCad board)
At the start: 2 copper layers, 156 x 116.5 mm, 82 parts

Commit message: Create right half schematic, successfully sync with new right half PCB!
Parts:
- added C1: 10μF, Capacitor_SMD:C_0603_1608Metric, F.Cu at (218.8, 161.0)
- added C2: 10μF, Capacitor_SMD:C_0603_1608Metric, F.Cu at (223.7, 159.6)
- added L1: 2.2μH, huntercook:L_CJIANG_FTC404030S_4.1x4.1x3.0_SMD, F.Cu at (220.4, 164.8)
- added R1: 470kΩ, Resistor_SMD:R_0603_1608Metric, F.Cu at (224.5, 161.9)
- added R2: 51kΩ, Resistor_SMD:R_0603_1608Metric, F.Cu at (225.2, 159.6)
- added U1: TLV61070ADBV, Package_TO_SOT_SMD:SOT-23-6, F.Cu at (224.4, 164.7)
- added U2: SN74LV1T126DBVR, Package_TO_SOT_SMD:SOT-23-5, F.Cu at (221.2, 160.4)
- CONN1: value (none) -> LCD HEADER
- JST1: value (none) -> Battery Connector
- LED1: value (none) -> Outer Bottom
- LED10, LED11, LED12, LED13, LED14, LED16, LED17, LED18, LED19, LED2, LED20, LED21, LED22, LED23, LED25, LED26, LED3, LED5, LED6, LED7, LED8, LED9: value (none) -> WS2812B-2020
- LED15: value (none) -> Far Thumb
- LED24: value (none) -> Inner Bottom
- LED27: value (none) -> Inner Top
- LED4: value (none) -> Outer Top
- MCU1: value (none) -> nice_nano
- PWR1: value (none) -> Power SW
- RE1: value (none) -> CKW12
- RST1: value (none) -> Reset SW
- S1, S10, S11, S12, S13, S14, S15, S16, S17, S18, S19, S2, S20, S21, S22, S23, S24, S25, S26, S27, S3, S4, S5, S6, S7, S8, S9: value (none) -> PG1316S
Connections:
- net BAT_P renamed /BAT_P
- net LED_1 renamed /LED_1
- net LED_10 renamed /LED_10
- net LED_11 renamed /LED_11
- net LED_12 renamed /LED_12
- net LED_13 renamed /LED_13
- net LED_14 renamed /LED_14
- net LED_15 renamed /LED_15
- net LED_16 renamed /LED_16
- net LED_17 renamed /LED_17
- net LED_18 renamed /LED_18
- net LED_19 renamed /LED_19
- net LED_2 renamed /LED_2
- net LED_20 renamed /LED_20
- net LED_21 renamed /LED_21
- net LED_22 renamed /LED_22
- net LED_23 renamed /LED_23
- net LED_24 renamed /LED_24
- net LED_25 renamed /LED_25
- net LED_26 renamed /LED_26
- net LED_27 renamed /LED_27
- net LED_3 renamed /LED_3
- net LED_4 renamed /LED_4
- net LED_5 renamed /LED_5
- net LED_6 renamed /LED_6
- net LED_7 renamed /LED_7
- net LED_8 renamed /LED_8
- net LED_9 renamed /LED_9
- net RST renamed /RST
- net mirror_far_fan renamed /far_fan
- net mirror_index_bottom renamed /index_bottom
- net mirror_index_home renamed /index_home
- net mirror_index_num renamed /index_num
- net mirror_index_top renamed /index_top
- net mirror_inner_bottom renamed /inner_bottom
- net mirror_inner_home renamed /inner_home
- net mirror_inner_num renamed /inner_num
- net mirror_inner_top renamed /inner_top
- net mirror_mid_fan renamed /mid_fan
- net mirror_middle_bottom renamed /middle_bottom
- net mirror_middle_home renamed /middle_home
- net mirror_middle_num renamed /middle_num
- net mirror_middle_top renamed /middle_top
- net mirror_near_fan renamed /near_fan
- net mirror_outer_bottom renamed /outer_bottom
- net mirror_outer_home renamed /outer_home
- net mirror_outer_num renamed /outer_num
- net mirror_outer_top renamed /outer_top
- net mirror_pinky_bottom renamed /pinky_bottom
- net mirror_pinky_home renamed /pinky_home
- net mirror_pinky_num renamed /pinky_num
- net mirror_pinky_top renamed /pinky_top
- net mirror_ring_bottom renamed /ring_bottom
- net mirror_ring_home renamed /ring_home
- net mirror_ring_num renamed /ring_num
- net mirror_ring_top renamed /ring_top
- net mirror_roller renamed /roller
- LED15 pad 3: LED_D5V -> /LED_D5V
- PWR1 pad 1: RAW -> unconnected-(PWR1-A-Pad1)
- PWR1 pad 3: (no net) -> RAW

Commit message: Fully route left half. Schematic and PCB both clean!
Parts:
- moved C2 2.73 mm to (223.6, 156.9)
- moved R2 2.73 mm to (225.1, 156.9)
- moved U2 2.73 mm to (221.2, 157.7)
- moved R1 2.73 mm to (224.4, 159.2)
- moved U1 2.73 mm to (224.3, 162.0)
- moved C1 2.73 mm to (218.7, 158.2)
- moved L1 2.73 mm to (220.3, 162.1)
Connections:
- MCU1 pad 15: LCD_DIN -> LCD_BL
- MCU1 pad 16: LCD_CLK -> LCD_DC
- MCU1 pad 17: LCD_DC -> LCD_CLK
- MCU1 pad 18: LCD_BL -> LCD_DIN
- PWR1 pad 1: unconnected-(PWR1-A-Pad1) -> RAW
- PWR1 pad 3: RAW -> unconnected-(PWR1-C-Pad3)
Routing:
- net /BAT_P: track 0.00 -> 24.1 mm, vias 0 -> 3
- net RAW: track 0.00 -> 21.6 mm, vias 0 -> 7
- net 5V: track 0.00 -> 6.04 mm, vias 0 -> 6
Other:
- copper layers 2 -> 6
