File: output/pcbs/toomanykeys_left_unrouted.kicad_pcb (KiCad board)
At the start: 2 copper layers, 156 x 116.5 mm, 82 parts

Commit message: Cleanup.
Parts:
- moved LED13 170.9 mm to (18.8, -4.82)
- moved LED14 170.9 mm to (17.8, -23.8)
- moved LED16 170.9 mm to (15.8, -61.7)
- moved MH7 170.9 mm to (136.9, 17.5)
- moved S6 170.9 mm to (17.9, -21.3)
- moved CONN1 170.9 mm to (122.6, -25.6)
- moved D1 170.9 mm to (51.6, 6.36)
- moved D10 170.9 mm to (45.6, 6.36)
- moved D11 170.9 mm to (63.6, 13.4)
- moved D12 170.9 mm to (45.6, 13.4)
- moved D13 170.9 mm to (69.6, 6.36)
- moved D14 170.9 mm to (69.6, 13.4)
- moved D2 170.9 mm to (33.6, 6.36)
- moved D3 170.9 mm to (51.6, 13.4)
- moved D4 170.9 mm to (33.6, 13.4)
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