File: output/pcbs/toomanykeys_right_unrouted.kicad_pcb (KiCad board)
At the start: 2 copper layers, 156 x 116.5 mm, 82 parts

Commit message: Cleanup.
Parts:
- moved CONN1 170.9 mm to (169.8, -25.6)
- moved JST1 170.9 mm to (157.8, 11.4)
- moved LCD1 170.9 mm to (169.8, -40.1)
- moved LED10 170.9 mm to (216.8, -29.1)
- moved LED11 170.9 mm to (216.8, -48.1)
- moved LED12 170.9 mm to (216.8, -67.1)
- moved LED13 170.9 mm to (208.8, 9.86)
- moved LED16 170.9 mm to (273.6, -4.82)
- moved LED17 170.9 mm to (274.6, -23.8)
- moved LED19 170.9 mm to (276.6, -61.7)
- moved LED24 170.9 mm to (197.8, -9.14)
- moved LED25 170.9 mm to (197.8, -28.1)
- moved LED26 170.9 mm to (197.8, -47.1)
- moved LED27 170.9 mm to (197.8, -66.1)
- moved LED9 170.9 mm to (216.8, -10.1)
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